Commit message: Update xacro files handing the robot and the table

File: lwr_simulation/model/urdf/robots/kuka_lwr.gzreferences.xacro (robot description, xacro)
@@ -1,10 +1,11 @@
 <?xml version="1.0"?>
-<robot xmlns:xacro="http://www.ros.org/wiki/xacro">
-	<xacro:macro name="kuka_lwr_gazebo" params="name">
-		<gazebo>
+<robot xmlns:xacro="http://ros.org/wiki/xacro">
+	<xacro:macro name="kuka_lwr_gz_references" params="name">
+		# this should be removed from here and if needed, be called from somewhere esle
+		<!--gazebo>
 			<plugin name="${name}_lwr_hw_sim" filename="liblwr_hw_gazebo_plugin.so">
 				<robotNamespace>${name}</robotNamespace>
 			</plugin>
-		</gazebo>
+		</gazebo-->
 		<gazebo reference="${name}_base_link">
 			<gravity>true</gravity>
