Commit message: Align the table, update the rviz.config

File: lwr_simulation/model/urdf/objects/table.xacro (robot description, xacro)
@@ -23,5 +23,5 @@
         </inertial>
         <visual>
-            <origin xyz="0.018511509179121 0.23251932391586 0" rpy="0 0 0" />
+            <origin xyz="-0.02 0.17 0" rpy="0 0 0" />
             <geometry>
                 <mesh filename="package://lwr_simulation/model/urdf/objects/meshes/table_base.STL" />
@@ -45,10 +45,10 @@
     <link name="table_top">
         <inertial>
-            <origin xyz="2.18575157973078E-16 0.0165 -1.11022302462516E-16" rpy="0 0 0" />
+            <origin xyz="0 0 0" rpy="0 0 0" />
             <mass value="27.72" />
             <inertia ixx="1.48091559" ixy="-4.70197740328915E-35" ixz="1.33744867033177E-16" iyy="4.025175" iyz="0" izz="2.54929059" />
         </inertial>
         <visual>
-            <origin xyz="0 -0.0165 0" rpy="0 0 0" />
+            <origin xyz="0 0 0" rpy="0 0 0" />
             <geometry>
                 <mesh filename="package://lwr_simulation/model/urdf/objects/meshes/table_top.STL" />
@@ -58,5 +58,11 @@
             </material>
         </visual>
-        <visual>
+        <collision>
+            <origin xyz="0 0 0" rpy="0 0 0" />
+            <geometry>
+                <mesh filename="package://lwr_simulation/model/urdf/objects/meshes/table_top.STL" />
+            </geometry>
+        </collision>
+        <!--visual>
             <origin xyz="0 ${t_thickness+rim_height/2} ${-t_height/2+rim_thickness/2}" rpy="0 0 0" />
             <geometry>
@@ -75,6 +81,6 @@
                 <color rgba="0.8 0.8 1 1" />
             </material>
-        </visual>
-        <collision>
+        </visual-->
+        <!--collision>
             <origin xyz="0 ${t_thickness+rim_height/2} ${-t_height/2+rim_thickness/2}" rpy="0 0 0" />
             <geometry>
@@ -87,14 +93,8 @@
                 <box size="${rim_thickness} ${rim_height} ${t_height}"/>
             </geometry>
-        </collision>
-        <collision>
-            <origin xyz="0 0 0" rpy="0 0 0" />
-            <geometry>
-                <mesh filename="package://lwr_simulation/model/urdf/objects/meshes/table_top.STL" />
-            </geometry>
-        </collision>
+        </collision-->
     </link>
     <joint name="j1" type="fixed">
-        <origin xyz="0 0 0.397575968372377" rpy="1.5707963267949 0 0" />
+        <origin xyz="0 0 0.38" rpy="1.5707963267949 0 0" />
         <parent link="table_base" />
         <child link="table_top" />
