Commit message: add gazebo plugin for publishing joint states

File: lwr_simulation/model/gzplugins/gzplugin_lwr_interface.xacro (robot description, xacro)
@@ -5,4 +5,14 @@
  xmlns:interface="http://playerstage.sourceforge.net/gazebo/xmlschema/#interface"
  xmlns:xacro="http://ros.org/wiki/xacro">
+<!-- macro to laod lwr joint interface -->
+<xacro:macro name="gzplugin_lwr_joint_interface" params="robot_components_namespace">
+    <gazebo>
+        <plugin name="gzplugin_lwr_joint_state_publisher" filename="libGazeboLwrJointStatePublisher.so">
+            <robot_components_namespace>
+                ${robot_components_namespace}
+            </robot_components_namespace>
+        </plugin>
+    </gazebo>
+</xacro:macro>
 <!-- macro to laod jaco control plugins -->
 <!--xacro:macro name="gzplugin_joint_control" params="robot_components_namespace trajectory_param_namespace">

File: lwr_simulation/model/lwr_on_table_gzplugins.xacro (robot description, xacro)
@@ -23,4 +23,9 @@
     </xacro:lwr_on_table>
     <!-- Attaching the gazebo plugings to the robot -->
+    <xacro:if value="true">
+        <xacro:include filename="$(find lwr_simulation)/model/gzplugins/gzplugin_lwr_interface.xacro"/>
+        <xacro:gzplugin_lwr_joint_interface robot_components_namespace="$(arg robot_components_namespace)"/>
+    </xacro:if>
+    <!-- Attaching the gazebo plugings to the robot -->
     <!--xacro:if value="$(arg use_ros_control)">
         <xacro:include filename="$(find lwr_simulation)/model/gzplugin_ros_control.urdf.xacro"/>
